Commit message: added object and env code

File: description/urdf/octopus_arm.urdf (robot description, URDF)
Before this commit: robot octopus_arm, 15 links, 14 joints
Joints:
- joint world_joint: origin xyz=-1.5 0 5.0 rpy=0 1.5708 0 -> xyz=-1.5 0 3.0 rpy=0 1.5708 0

Commit message: added training code

File: description/urdf/octopus_arm.urdf (robot description, URDF)
Before this commit: robot octopus_arm, 15 links, 14 joints
Links:
- link Plane_001: mass 0.05 -> 0.5
- link Plane_002: mass 0.05 -> 0.5
- link Plane_003: mass 0.05 -> 0.5
- link Plane_004: mass 0.05 -> 0.5
- link Plane_005: mass 0.05 -> 0.5
- link Plane_006: mass 0.05 -> 0.5
- link Plane_007: mass 0.05 -> 0.5
- link Plane_008: mass 0.05 -> 0.5
- link Plane_009: mass 0.05 -> 0.5
- link Plane_010: mass 0.05 -> 0.5
- link Plane_011: mass 0.05 -> 0.5
- link Plane_012: mass 0.05 -> 0.5
Joints:
- joint world_joint: origin xyz=-1.5 0 3.0 rpy=0 1.5708 0 -> xyz=-1.5 0 4.0 rpy=0 1.5708 0

Commit message: training

File: description/urdf/octopus_arm.urdf (robot description, URDF)
Before this commit: robot octopus_arm, 15 links, 14 joints
Joints:
- joint world_joint: origin xyz=-1.5 0 4.0 rpy=0 1.5708 0 -> xyz=0.0 0 6.0 rpy=0 1.7708 0

Commit message: fixed bugs for obs and fruit and all   env.py

File: description/urdf/octopus_arm.urdf (robot description, URDF)
Before this commit: robot octopus_arm, 15 links, 14 joints
Joints:
- joint world_joint: origin xyz=0.0 0 6.0 rpy=0 1.7708 0 -> xyz=0.0 0 5.0 rpy=0 1.7708 0
